File: PCB_UPDI_for_AE-CH9102F.kicad_pcb (KiCad board)
At the start: 2 copper layers, 22.9 x 17.8 mm, 8 parts, among them J1 AE-CH9102F, J2 UPDI, J3 TTL Serial, J4 RTS / DTR, SW1 UPDI / Serial, SW2 Power

Commit message: Rev. 2
Implement auto switching between the UPDI mode and the UART mode.
Parts:
- removed SW1: UPDI / Serial, Connector_PinHeader_2.54mm:PinHeader_1x03_P2.54mm_Vertical
- added D2: BAT43, Diode_THT:D_DO-35_SOD27_P2.54mm_Vertical_KathodeUp, F.Cu at (96.5, 63.5)
- added Q1: BSS138, Package_TO_SOT_SMD:SOT-23, F.Cu at (87.6, 68.6)
- added Q2: BSS84, Package_TO_SOT_SMD:SOT-23, F.Cu at (91.8, 68.6)
- added R2: 100k, Resistor_THT:R_Axial_DIN0204_L3.6mm_D1.6mm_P2.54mm_Vertical, F.Cu at (90.2, 66.0)
- D1: value D_Schottky -> BAT43; footprint Diode_THT:D_A-405_P2.54mm_Vertical_KathodeUp -> Diode_THT:D_DO-35_SOD27_P2.54mm_Vertical_KathodeUp
- moved J4 2.56 mm to (83.8, 63.5)
Connections:
- J2 pad 4: /RxD -> /UPDI
- R1 pad 1: Net-(SW1-C) -> /UPDI
Routing:
- net +5V: track 8.72 -> 31.0 mm
- net /UPDI: track 0.00 -> 15.9 mm
- net /RxD (TTL): track 15.2 -> 3.59 mm
- net RTS: track 12.1 -> 18.8 mm
- net /RxD: track 17.3 -> 11.0 mm
- net Net-(D2-A): track 0.00 -> 5.61 mm
- net Net-(SW1-C): track 4.86 -> 0.00 mm
- net GND: track 0.00 -> 4.34 mm
- net /RTS/DTR: track 11.2 -> 13.8 mm
Other:
- board text added: "NC"
- board text added: "UPDI Adapter for AE-CH9102F"
- board text removed: "Data"

Commit message: Update for Rev. 3
* Use 74LVC1G3157.
* Use SMD devices.
Parts:
- removed D2: BAT43, Diode_THT:D_DO-35_SOD27_P2.54mm_Vertical_KathodeUp
- removed Q1: BSS138, Package_TO_SOT_SMD:SOT-23
- removed Q2: BSS84, Package_TO_SOT_SMD:SOT-23
- added U1: 74LVC1G3157, Package_TO_SOT_SMD:SOT-23-6, F.Cu at (88.9, 68.6)
- D1: value BAT43 -> BAT43WS; footprint Diode_THT:D_DO-35_SOD27_P2.54mm_Vertical_KathodeUp -> Diode_SMD:D_0603_1608Metric
- R1, R2: footprint Resistor_THT:R_Axial_DIN0204_L3.6mm_D1.6mm_P2.54mm_Vertical -> Resistor_SMD:R_0603_1608Metric
- moved R2 1.91 mm to (92.1, 66.0)
- moved D1 1.91 mm to (88.3, 72.4)
- moved R1 1.91 mm to (92.1, 72.4)
Routing:
- net /RxD (TTL): track 3.59 -> 14.2 mm
- net +5V: track 31.0 -> 38.4 mm
- net Net-(D2-A): track 5.61 -> 0.00 mm
- net GND: track 4.34 -> 8.80 mm, vias 0 -> 1
- net RTS: track 18.8 -> 15.2 mm
- net /UPDI: track 15.9 -> 17.3 mm
- net /RxD: track 11.0 -> 11.6 mm
